Commit message: modify for damping

File: crane_x7_description/urdf/crane_x7_arm.xacro (robot description, xacro)
@@ -84,5 +84,5 @@
       <parent link="${NAME_LINK_BASE}"/>
       <child link="${NAME_LINK_1}"/>
-      <dynamics damping="1.0e-6" friction="2.0e-1"/>
+      <dynamics damping="1.0e-6" friction="0"/>
     </joint>
     <!-- For gazebo simulation -->
@@ -142,5 +142,5 @@
       <parent link="${NAME_LINK_1}"/>
       <child link="${NAME_LINK_2}"/>
-      <dynamics damping="1.0e-6" friction="2.0e-1"/>
+      <dynamics damping="1.0e-6" friction="0"/>
     </joint>
     <!-- For gazebo simulation -->
@@ -227,5 +227,5 @@
       <parent link="${NAME_LINK_2}"/>
       <child link="${NAME_LINK_3}"/>
-      <dynamics damping="1.0e-6" friction="2.0e-1"/>
+      <dynamics damping="1.0e-6" friction="0"/>
     </joint>
     <!-- For gazebo simulation -->
@@ -278,5 +278,5 @@
       <parent link="${NAME_LINK_3}"/>
       <child link="${NAME_LINK_4}"/>
-      <dynamics damping="1.0e-6" friction="2.0e-1"/>
+      <dynamics damping="1.0e-6" friction="0"/>
     </joint>
     <!-- For gazebo simulation -->
@@ -360,5 +360,5 @@
       <parent link="${NAME_LINK_4}"/>
       <child link="${NAME_LINK_5}"/>
-      <dynamics damping="1.0e-6" friction="2.0e-1"/>
+      <dynamics damping="1.0e-6" friction="0"/>
     </joint>
     <!-- For gazebo simulation -->
@@ -413,5 +413,5 @@
       <parent link="${NAME_LINK_5}"/>
       <child link="${NAME_LINK_6}"/>
-      <dynamics damping="1.0e-6" friction="2.0e-1"/>
+      <dynamics damping="1.0e-6" friction="0"/>
     </joint>
     <!-- For gazebo simulation -->
@@ -461,5 +461,5 @@
       <parent link="${NAME_LINK_6}"/>
       <child link="${end_effector_base_link}"/>
-      <dynamics damping="1.0e-6" friction="2.0e-1"/>
+      <dynamics damping="1.0e-6" friction="0"/>
     </joint>
     <!-- For gazebo simulation -->
