Commit message: udpate for noetic

File: crane_x7_description/urdf/crane_x7.urdf.xacro (robot description, xacro)
@@ -21,5 +21,5 @@
        allows accessing different operational areas, e.g. left-handed vs.
        right-handed robots. -->
-  <crane_x7 parent="base_link"
+  <xacro:crane_x7 parent="base_link"
               base_color="red"
               shoulder_color="white"
@@ -38,4 +38,4 @@
               use_effort_gripper="$(arg use_effort_gripper)">
     <origin xyz="0 0 0"/>
-  </crane_x7>
+  </xacro:crane_x7>
 </robot>

File: crane_x7_description/urdf/crane_x7.xacro (robot description, xacro)
@@ -42,12 +42,12 @@
     <!-- Mounting plate
          (Root of the manipulator's TF tree) -->
-    <crane_x7_mounting_plate
+    <xacro:crane_x7_mounting_plate
         parent="${parent}"
         name="crane_x7_mounting_plate"
         color="silver">
       <xacro:insert_block name="origin"/>
-    </crane_x7_mounting_plate>
+    </xacro:crane_x7_mounting_plate>
     <!-- Arm -->
-    <crane_x7_arm
+    <xacro:crane_x7_arm
         parent="crane_x7_mounting_plate_link"
         end_effector_base_link="crane_x7_gripper_base_link"
@@ -66,7 +66,7 @@
         logos_definition="${logos_definition}">
       <origin xyz="0 0 ${MOUNTING_PLATE_THICKNESS}" rpy="0 0 0"/>
-    </crane_x7_arm>
+    </xacro:crane_x7_arm>
     <!-- End effector -->
-    <crane_x7_wide_two_finger_gripper
+    <xacro:crane_x7_wide_two_finger_gripper
         name="crane_x7_gripper"
         color="${hand_color}"

File: crane_x7_description/urdf/crane_x7_arm.xacro (robot description, xacro)
@@ -84,5 +84,5 @@
       <parent link="${NAME_LINK_BASE}"/>
       <child link="${NAME_LINK_1}"/>
-      <dynamics damping="1.0e-6" friction="0"/>
+      <dynamics damping="1.0e-6" friction="2.0e-1"/>
     </joint>
     <!-- For gazebo simulation -->
@@ -142,5 +142,5 @@
       <parent link="${NAME_LINK_1}"/>
       <child link="${NAME_LINK_2}"/>
-      <dynamics damping="1.0e-6" friction="0"/>
+      <dynamics damping="1.0e-6" friction="2.0e-1"/>
     </joint>
     <!-- For gazebo simulation -->
@@ -199,4 +199,11 @@
         <material name="${shoulder_joint_cover_color}"/>
       </visual>
+      <collision>
+        <origin xyz="0 0 0" rpy="-${M_PI/2} 0 0"/>
+        <geometry>
+          <mesh filename="package://crane_x7_description/meshes/visual/joint_cover.stl"
+              scale="1 1 1"/>
+        </geometry>
+      </collision>
     </link>
     <!-- crane_x7_joint_cover_2_r -->
@@ -216,4 +223,11 @@
         <material name="${shoulder_joint_cover_color}"/>
       </visual>
+      <collision>
+        <origin xyz="0 0 0" rpy="${M_PI/2} 0 0"/>
+        <geometry>
+          <mesh filename="package://crane_x7_description/meshes/visual/joint_cover.stl"
+              scale="1 1 1"/>
+        </geometry>
+      </collision>
     </link>
     <!-- crane_x7_joint_3 -->
@@ -227,5 +241,5 @@
       <parent link="${NAME_LINK_2}"/>
       <child link="${NAME_LINK_3}"/>
-      <dynamics damping="1.0e-6" friction="0"/>
+      <dynamics damping="1.0e-6" friction="2.0e-1"/>
     </joint>
     <!-- For gazebo simulation -->
@@ -278,5 +292,5 @@
       <parent link="${NAME_LINK_3}"/>
       <child link="${NAME_LINK_4}"/>
-      <dynamics damping="1.0e-6" friction="0"/>
+      <dynamics damping="1.0e-6" friction="2.0e-1"/>
     </joint>
     <!-- For gazebo simulation -->
@@ -335,4 +349,11 @@
         <material name="${elbow_joint_cover_color}"/>
       </visual>
+      <collision>
+        <origin xyz="0 0 0" rpy="-${M_PI/2} 0 0"/>
+        <geometry>
+          <mesh filename="package://crane_x7_description/meshes/visual/joint_cover.stl"
+              scale="1 1 1"/>
+        </geometry>
+      </collision>
     </link>
     <!-- crane_x7_joint_cover_4_r -->
@@ -352,4 +373,11 @@
         <material name="${elbow_joint_cover_color}"/>
       </visual>
+      <collision>
+        <origin xyz="0 0 0" rpy="${M_PI/2} 0 0"/>
+        <geometry>
+          <mesh filename="package://crane_x7_description/meshes/visual/joint_cover.stl"
+              scale="1 1 1"/>
+        </geometry>
+      </collision>
     </link>
     <!-- crane_x7_joint_5 -->
@@ -357,8 +385,8 @@
       <origin xyz="0 0 0.121" rpy="0 0 0"/>
       <axis xyz="0 0 1"/>
-      <limit effort="4.0" velocity="${joints_vlimit}" lower="-2.77343" upper="1.51403"/>
+      <limit effort="4.0" velocity="${joints_vlimit}" lower="-2.77343" upper="2.77343"/>
       <parent link="${NAME_LINK_4}"/>
       <child link="${NAME_LINK_5}"/>
-      <dynamics damping="1.0e-6" friction="0"/>
+      <dynamics damping="1.0e-6" friction="2.0e-1"/>
     </joint>
     <!-- For gazebo simulation -->
@@ -403,5 +431,5 @@
     <!-- logo -->
     <xacro:include filename="${logos_definition}"/>
-    <crane_x7_logos
+    <xacro:crane_x7_logos
       parent="${NAME_LINK_5}"
       name="${NAME_LOGO}"/>
@@ -413,5 +441,5 @@
       <parent link="${NAME_LINK_5}"/>
       <child link="${NAME_LINK_6}"/>
-      <dynamics damping="1.0e-6" friction="0"/>
+      <dynamics damping="1.0e-6" friction="2.0e-1"/>
     </joint>
     <!-- For gazebo simulation -->
@@ -461,5 +489,5 @@
       <parent link="${NAME_LINK_6}"/>
       <child link="${end_effector_base_link}"/>
-      <dynamics damping="1.0e-6" friction="0"/>
+      <dynamics damping="1.0e-6" friction="2.0e-1"/>
     </joint>
     <!-- For gazebo simulation -->

File: crane_x7_description/urdf/crane_x7_rt_logos.xacro (robot description, xacro)
@@ -14,4 +14,11 @@
         </material>
       </visual>
+      <collision>
+        <origin xyz="0 0 0" rpy="-${M_PI/2} ${M_PI/2} 0"/>
+        <geometry>
+          <mesh filename="package://crane_x7_description/meshes/visual/rtcorp_logo_name.stl"
+              scale="1 1 1"/>
+        </geometry>
+      </collision>
     </link>
     <joint name="${name}_logo_text_l_joint" type="fixed">
@@ -30,4 +37,11 @@
         <material name="logo_red"/>
       </visual>
+      <collision>
+        <origin xyz="0 0 0" rpy="-${M_PI/2} ${M_PI/2} 0"/>
+        <geometry>
+          <mesh filename="package://crane_x7_description/meshes/visual/rtcorp_logo_rabbit.stl"
+              scale="1 1 1"/>
+        </geometry>
+      </collision>
     </link>
     <joint name="${name}_logo_symbol_l_joint" type="fixed">
@@ -46,4 +60,11 @@
         <material name="logo_red"/>
       </visual>
+      <collision>
+        <origin xyz="0 0 0" rpy="${M_PI/2} -${M_PI/2} 0"/>
+        <geometry>
+          <mesh filename="package://crane_x7_description/meshes/visual/rtcorp_logo_name.stl"
+              scale="1 1 1"/>
+        </geometry>
+      </collision>
     </link>
     <joint name="${name}_logo_text_r_joint" type="fixed">
@@ -62,4 +83,11 @@
         <material name="logo_red"/>
       </visual>
+      <collision>
+        <origin xyz="0 0 0" rpy="${M_PI/2} -${M_PI/2} 0"/>
+        <geometry>
+          <mesh filename="package://crane_x7_description/meshes/visual/rtcorp_logo_rabbit.stl"
+              scale="1 1 1"/>
+        </geometry>
+      </collision>
     </link>
     <joint name="${name}_logo_symbol_r_joint" type="fixed">

File: crane_x7_description/urdf/crane_x7_wide_two_finger_gripper.xacro (robot description, xacro)
@@ -121,5 +121,5 @@
     <!-- For gazebo simulation -->
     <gazebo>
-      <plugin name="crane_x7_gripper_mimic_joint" filename="libroboticsgroup_gazebo_mimic_joint_plugin.so">
+      <plugin name="crane_x7_gripper_mimic_joint" filename="libroboticsgroup_upatras_gazebo_mimic_joint_plugin.so">
         <joint>${name}_finger_a_joint</joint>
         <mimicJoint>${name}_finger_b_joint</mimicJoint>
